File: kicad/GameHardware/GameHardware.kicad_sch (KiCad schematic)
At the start: 9 parts, among them U1 MAX7219, U2 ATmega328P-P, U4 HDSP-7403, U5 HDSP-7403, U6 HDSP-7403, U7 HDSP-7403, U8 HDSP-7403, U9 HDSP-7403

Commit message: pill
Parts:
- removed U4: HDSP-7403, Display_7Segment:Sx39-1xxxxx, symbol Display_Character:HDSP-7403
- added U10: HDSP-7403, Display_7Segment:Sx39-1xxxxx, symbol Display_Character:HDSP-7403
Connections:
- net A: now also U5.10 (A), U6.10 (A), U7.10 (A), U8.10 (A), U9.10 (A), U10.10 (A)
- net B: now also U5.9 (B), U6.9 (B), U7.9 (B), U8.9 (B), U9.9 (B), U10.9 (B)
- net C: now also U5.7 (C), U6.7 (C), U7.7 (C), U8.7 (C), U9.7 (C), U10.7 (C)
- net D: now also U5.5 (D), U6.5 (D), U7.5 (D), U8.5 (D), U9.5 (D), U10.5 (D)
- net DIG0: now also U5.3 (GND), U5.8 (GND)
- net DIG1: now also U6.3 (GND), U6.8 (GND)
- net DIG2: now also U7.3 (GND), U7.8 (GND)
- net DIG3: now also U8.3 (GND), U8.8 (GND)
- net DIG4: now also U9.3 (GND), U9.8 (GND)
- net DIG5: now also U10.3 (GND), U10.8 (GND)
- net DP: now also U5.6 (DP), U6.6 (DP), U7.6 (DP), U8.6 (DP), U9.6 (DP), U10.6 (DP)
- net E: now also U5.4 (E), U6.4 (E), U7.4 (E), U8.4 (E), U9.4 (E), U10.4 (E)
- net F: now also U5.2 (F), U6.2 (F), U7.2 (F), U8.2 (F), U9.2 (F), U10.2 (F)
- net G: now also U5.1 (G), U6.1 (G), U7.1 (G), U8.1 (G), U9.1 (G), U10.1 (G)

Commit message: more kicad
Parts:
- added D1, D10, D11, D12, D13, D14, D15, D16, D2, D3, D4, D5, D6, D7, D8, D9: LED, LED_THT:LED_D3.0mm_Clear, symbol Device:LED
- added J5: USB_B, Connector_USB:USB_B_Lumberg_2411_02_Horizontal, symbol Connector:USB_B
- added J6: ISP header, Connector_PinHeader_2.54mm:PinHeader_2x03_P2.54mm_Horizontal, symbol Connector_Generic:Conn_02x03_Odd_Even
- R1: value R -> 10k; footprint (none) -> Resistor_THT:R_Axial_DIN0204_L3.6mm_D1.6mm_P7.62mm_Horizontal
Connections:
- net A: now also D1.2 (A), D9.2 (A)
- net B: now also D10.2 (A), D2.2 (A)
- net C: now also D11.2 (A), D3.2 (A)
- net D: now also D12.2 (A), D4.2 (A)
- net DIG6: now also D1.1 (K), D2.1 (K), D3.1 (K), D4.1 (K), D5.1 (K), D6.1 (K), D7.1 (K), D8.1 (K)
- net DIG7: now also D10.1 (K), D11.1 (K), D12.1 (K), D13.1 (K), D14.1 (K), D15.1 (K), D16.1 (K), D9.1 (K)
- net DP: now also D16.2 (A), D8.2 (A)
- net E: now also D13.2 (A), D5.2 (A)
- net F: now also D14.2 (A), D15.2 (A), D6.2 (A), D7.2 (A)
- net GND: now also U2.22 (GND), U2.8 (GND), J5.4 (GND), J5.5 (Shield), J6.6 (Pin_6)
- net MOSI: now reaches U1.1 (DIN)
- net MOSI: now also U2.17 (PB3), J6.4 (Pin_4)
- net LOAD: now reaches U1.12 (LOAD)
- net LOAD: now also U2.16 (PB2)
- net SCK: now reaches U1.13 (CLK)
- net SCK: now also U2.19 (PB5), J6.3 (Pin_3)
- net 5V: now reaches U1.19 (V+)
- net 5V: now also U2.7 (VCC)
- net MISO: now reaches U2.18 (PB4)
- net MISO: now also J6.1 (Pin_1)
- new net +5V: J5.1 (VBUS), J6.2 (Pin_2)
- new net Reset: J6.5 (Pin_5)
