File: kicad/Game_project/game.kicad_pcb (KiCad board)
At the start: 2 copper layers, 27 parts, among them J5 USB_B, J6 ISP header, U1 MAX7219, U10 HDSP-7403, U2 ATmega328P-P, U5 HDSP-7403, U6 HDSP-7403, U7 HDSP-7403, U8 HDSP-7403, U9 HDSP-7403

Commit message: started i pcb
Parts:
- moved U9 162.0 mm to (228.1, 109.3), turned to 90 degrees
- moved U10 146.9 mm to (228.2, 98.7), turned to 90 degrees
Other:
- board outline added: 136.8 x 99.6 mm
Changed lines of the file:
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@@
 	(footprint "Display_7Segment:Sx39-1xxxxx"
 		(layer "F.Cu")
-		(at 95.03 36.795)
+		(at 228.1975 98.7325 90)
 		(descr "Single digit 7 segment LED display in red, yellow or green colour http://www.kingbrightusa.com/images/catalog/SPEC/sa39-11ewa.pdf")
 		(tags "One digit LED 7 segment SA39-11 SC39-11 SA39-12 SC39-12")
 		(property "Reference" "U10"
-			(at 3.81 -2.54 0)
+			(at 3.81 -2.54 90)
 			(layer "F.SilkS")
 			(effects
@@
 		)
 		(property "Value" "HDSP-7403"
-			(at 2.54 12.7 0)
+			(at 2.54 12.7 90)
 			(layer "F.Fab")
 			(effects
@@
 		)
 		(property "Datasheet" "https://docs.broadcom.com/docs/AV02-2553EN"
-			(at 0 0 0)
+			(at 0 0 90)
 			(unlocked yes)
 			(layer "F.Fab")
@@
 		)
 		(property "Description" "One digit 7 segment yellow, common cathode"
-			(at 0 0 0)
+			(at 0 0 90)
 			(unlocked yes)
 			(layer "F.Fab")
@@
 		)
 		(fp_line
-			(start -1.66 -0.69)
-			(end -1.66 -1.89)
+			(start 8.92 -1.53)
+			(end -1.3 -1.53)
 			(stroke
 				(width 0.12)
@@
 		)
 		(fp_line
-			(start -1.3 11.69)
-			(end 8.92 11.69)
+			(start -1.66 -0.69)
+			(end -1.66 -1.89)
 			(stroke
 				(width 0.12)
@@
 		)
 		(fp_line
-			(start 8.92 -1.53)
-			(end -1.3 -1.53)
+			(start 8.92 11.69)
+			(end 8.92 -1.53)
 			(stroke
 				(width 0.12)
@@
 		)
 		(fp_line
-			(start 8.92 11.69)
-			(end 8.92 -1.53)
+			(start -1.3 11.69)
+			(end 8.92 11.69)
 			(stroke
 				(width 0.12)
@@
 		)
 		(fp_line
-			(start -1.44 -1.67)
-			(end 9.06 -1.67)
+			(start 9.06 -1.67)
+			(end 9.06 11.83)
 			(stroke
 				(width 0.05)
@@
 		)
 		(fp_line
-			(start -1.44 11.83)
-			(end -1.44 -1.67)
+			(start -1.44 -1.67)
+			(end 9.06 -1.67)
 			(stroke
 				(width 0.05)
@@
 		)
 		(fp_line
-			(start 9.06 -1.67)
-			(end 9.06 11.83)
+			(start 9.06 11.83)
+			(end -1.44 11.83)
 			(stroke
 				(width 0.05)
@@
 		)
 		(fp_line
-			(start 9.06 11.83)
-			(end -1.44 11.83)
+			(start -1.44 11.83)
+			(end -1.44 -1.67)
 			(stroke
 				(width 0.05)
@@
 		)
 		(fp_line
-			(start -1.19 -0.42)
-			(end -0.19 -1.42)
+			(start 8.81 -1.42)
+			(end 8.81 11.58)
 			(stroke
 				(width 0.1)
@@
 		)
 		(fp_line
-			(start -1.19 11.58)
-			(end -1.19 -0.42)
+			(start -0.19 -1.42)
+			(end 8.81 -1.42)
 			(stroke
 				(width 0.1)
@@
 		)
 		(fp_line
-			(start -0.19 -1.42)
-			(end 8.81 -1.42)
+			(start -1.19 -0.42)
+			(end -0.19 -1.42)
 			(stroke
 				(width 0.1)
@@
 		)
 		(fp_line
-			(start 8.81 -1.42)
-			(end 8.81 11.58)
+			(start 8.81 11.58)
+			(end -1.19 11.58)
 			(stroke
 				(width 0.1)
@@
 		)
 		(fp_line
-			(start 8.81 11.58)
-			(end -1.19 11.58)
+			(start -1.19 11.58)
+			(end -1.19 -0.42)
 			(stroke
 				(width 0.1)
@@
 		)
 		(fp_text user "${REFERENCE}"
-			(at 3.81 5.08 0)
+			(at 3.81 5.08 90)
 			(layer "F.Fab")
 			(effects
@@
 		)
 		(pad "1" thru_hole rect
-			(at 0 0)
+			(at 0 0 90)
 			(size 1.7 1.7)
 			(drill 1)
@@
 		)
 		(pad "2" thru_hole circle
-			(at 0 2.54)
+			(at 0 2.54 90)
 			(size 1.7 1.7)
 			(drill 1)
@@
 		)
 		(pad "3" thru_hole circle
-			(at 0 5.08)
+			(at 0 5.08 90)
 			(size 1.7 1.7)
 			(drill 1)
@@
 		)
 		(pad "4" thru_hole circle
-			(at 0 7.62)
+			(at 0 7.62 90)
 			(size 1.7 1.7)
 			(drill 1)
@@
 		)
 		(pad "5" thru_hole circle
-			(at 0 10.16)
+			(at 0 10.16 90)
 			(size 1.7 1.7)
 			(drill 1)
@@
 		)
 		(pad "6" thru_hole circle
-			(at 7.62 10.16)
+			(at 7.62 10.16 90)
 			(size 1.7 1.7)
 			(drill 1)
@@
 		)
 		(pad "7" thru_hole circle
-			(at 7.62 7.62)
+			(at 7.62 7.62 90)
 			(size 1.7 1.7)
 			(drill 1)
@@
 		)
 		(pad "8" thru_hole circle
-			(at 7.62 5.08)
+			(at 7.62 5.08 90)
 			(size 1.7 1.7)
 			(drill 1)
@@
 		)
 		(pad "9" thru_hole circle
-			(at 7.62 2.54)
+			(at 7.62 2.54 90)
 			(size 1.7 1.7)
 			(drill 1)
@@
 		)
 		(pad "10" thru_hole circle
-			(at 7.62 0)
+			(at 7.62 0 90)
 			(size 1.7 1.7)
 			(drill 1)
@@
 	(footprint "Display_7Segment:Sx39-1xxxxx"
 		(layer "F.Cu")
-		(at 83.225 36.795)
+		(at 228.1475 109.2825 90)
 		(descr "Single digit 7 segment LED display in red, yellow or green colour http://www.kingbrightusa.com/images/catalog/SPEC/sa39-11ewa.pdf")
 		(tags "One digit LED 7 segment SA39-11 SC39-11 SA39-12 SC39-12")
 		(property "Reference" "U9"
-			(at 3.81 -2.54 0)
+			(at 3.81 -2.54 90)
 			(layer "F.SilkS")
 			(effects
@@
 		)
 		(property "Value" "HDSP-7403"
-			(at 2.54 12.7 0)
+			(at 2.54 12.7 90)
 			(layer "F.Fab")
 			(effects
@@
 		)
 		(property "Datasheet" "https://docs.broadcom.com/docs/AV02-2553EN"
-			(at 0 0 0)
+			(at 0 0 90)
 			(unlocked yes)
 			(layer "F.Fab")
@@
 		)
 		(property "Description" "One digit 7 segment yellow, common cathode"
-			(at 0 0 0)
+			(at 0 0 90)
 			(unlocked yes)
 			(layer "F.Fab")
@@
 		)
 		(fp_line
-			(start -1.66 -0.69)
-			(end -1.66 -1.89)
+			(start 8.92 -1.53)
+			(end -1.3 -1.53)
 			(stroke
 				(width 0.12)
@@
 		)
 		(fp_line
-			(start -1.3 11.69)
-			(end 8.92 11.69)
+			(start -1.66 -0.69)
+			(end -1.66 -1.89)
 			(stroke
 				(width 0.12)
@@
 		)
 		(fp_line
-			(start 8.92 -1.53)
-			(end -1.3 -1.53)
+			(start 8.92 11.69)
+			(end 8.92 -1.53)
 			(stroke
 				(width 0.12)
@@
 		)
 		(fp_line
-			(start 8.92 11.69)
-			(end 8.92 -1.53)
+			(start -1.3 11.69)
+			(end 8.92 11.69)
 			(stroke
 				(width 0.12)
@@
 		)
 		(fp_line
-			(start -1.44 -1.67)
-			(end 9.06 -1.67)
+			(start 9.06 -1.67)
+			(end 9.06 11.83)
 			(stroke
 				(width 0.05)
@@
 		)
 		(fp_line
-			(start -1.44 11.83)
-			(end -1.44 -1.67)
+			(start -1.44 -1.67)
+			(end 9.06 -1.67)
 			(stroke
 				(width 0.05)
@@
 		)
 		(fp_line
-			(start 9.06 -1.67)
-			(end 9.06 11.83)
+			(start 9.06 11.83)
+			(end -1.44 11.83)
 			(stroke
 				(width 0.05)
@@
 		)
 		(fp_line
-			(start 9.06 11.83)
-			(end -1.44 11.83)
+			(start -1.44 11.83)
+			(end -1.44 -1.67)
 			(stroke
 				(width 0.05)
@@
 		)
 		(fp_line
-			(start -1.19 -0.42)
-			(end -0.19 -1.42)
+			(start 8.81 -1.42)
+			(end 8.81 11.58)
 			(stroke
 				(width 0.1)
@@
 		)
 		(fp_line
-			(start -1.19 11.58)
-			(end -1.19 -0.42)
+			(start -0.19 -1.42)
+			(end 8.81 -1.42)
 			(stroke
 				(width 0.1)
@@
 		)
 		(fp_line
-			(start -0.19 -1.42)
-			(end 8.81 -1.42)
+			(start -1.19 -0.42)
+			(end -0.19 -1.42)
 			(stroke
 				(width 0.1)
@@
 		)
 		(fp_line
-			(start 8.81 -1.42)
-			(end 8.81 11.58)
+			(start 8.81 11.58)
+			(end -1.19 11.58)
 			(stroke
 				(width 0.1)
@@
 		)
 		(fp_line
-			(start 8.81 11.58)
-			(end -1.19 11.58)
+			(start -1.19 11.58)
+			(end -1.19 -0.42)
 			(stroke
 				(width 0.1)
@@
 		)
 		(fp_text user "${REFERENCE}"
-			(at 3.81 5.08 0)
+			(at 3.81 5.08 90)
 			(layer "F.Fab")
 			(effects
@@
 		)
 		(pad "1" thru_hole rect
-			(at 0 0)
+			(at 0 0 90)
 			(size 1.7 1.7)
 			(drill 1)
@@
 		)
 		(pad "2" thru_hole circle
-			(at 0 2.54)
+			(at 0 2.54 90)
 			(size 1.7 1.7)
 			(drill 1)
@@
 		)
 		(pad "3" thru_hole circle
-			(at 0 5.08)
+			(at 0 5.08 90)
 			(size 1.7 1.7)
 			(drill 1)
@@
 		)
 		(pad "4" thru_hole circle
-			(at 0 7.62)
+			(at 0 7.62 90)
 			(size 1.7 1.7)
 			(drill 1)
@@
 		)
 		(pad "5" thru_hole circle
-			(at 0 10.16)
+			(at 0 10.16 90)
 			(size 1.7 1.7)
 			(drill 1)
@@
 		)
 		(pad "6" thru_hole circle
-			(at 7.62 10.16)
+			(at 7.62 10.16 90)
 			(size 1.7 1.7)
 			(drill 1)
@@
 		)
 		(pad "7" thru_hole circle
-			(at 7.62 7.62)
+			(at 7.62 7.62 90)
 			(size 1.7 1.7)
 			(drill 1)
@@
 		)
 		(pad "8" thru_hole circle
-			(at 7.62 5.08)
+			(at 7.62 5.08 90)
 			(size 1.7 1.7)
 			(drill 1)
@@
 		)
 		(pad "9" thru_hole circle
-			(at 7.62 2.54)
+			(at 7.62 2.54 90)
 			(size 1.7 1.7)
 			(drill 1)
@@
 		)
 		(pad "10" thru_hole circle
-			(at 7.62 0)
+			(at 7.62 0 90)
 			(size 1.7 1.7)
 			(drill 1)
@@
 		)
 	)
+	(gr_rect
+		(start 109.925 50.45)
+		(end 246.675 150.1)
+		(stroke
+			(width 0.2)
+			(type solid)
+		)
+		(fill no)
+		(layer "Edge.Cuts")
+	)
 	(embedded_fonts no)

Commit message: snart klar i kicad de ska bara rotas
Parts:
- added J3: Conn_01x05_Socket, Connector_PinSocket_2.54mm:PinSocket_1x05_P2.54mm_Vertical, F.Cu at (246.2, 105.6)
- added J4: Conn_01x05_Socket, Connector_PinSocket_2.54mm:PinSocket_1x05_P2.54mm_Vertical, F.Cu at (104.5, 94.7)
- added R2: 10k, Resistor_THT:R_Axial_DIN0204_L3.6mm_D1.6mm_P7.62mm_Horizontal, F.Cu at (177.2, 145.0)
- added R3: 10k, Resistor_THT:R_Axial_DIN0204_L3.6mm_D1.6mm_P7.62mm_Horizontal, F.Cu at (166.2, 145.2)
- added RESET: SW_pin12, Button_Switch_THT:SW_PUSH-12mm_Wuerth-430476085716, F.Cu at (147.5, 123.0)
- added WHEEL: SW_pin12, Button_Switch_THT:SW_PUSH-12mm_Wuerth-430476085716, F.Cu at (147.5, 136.5)
- U1: footprint Package_DIP:DIP-24_18.0mmx34.29mm_W15.24mm -> Package_DIP:DIP-28_W7.62mm
- moved U2 175.6 mm to (210.9, 55.9), turned to -90 degrees
- moved U7 171.4 mm to (219.9, 97.5), turned to 90 degrees
- moved U8 164.7 mm to (219.7, 108.5), turned to 90 degrees
- moved D14 158.3 mm to (227.2, 123.5), turned to 90 degrees
- moved D13 146.8 mm to (227.8, 78.8), turned to 90 degrees
- moved J6 134.2 mm to (219.2, 65.2), turned to 90 degrees
- moved D11 125.8 mm to (198.5, 97.8)
- moved D12 125.6 mm to (198.5, 102.2)
- moved U1 125.6 mm to (172.2, 55.6), turned to -90 degrees
- moved D10 118.0 mm to (177.5, 120.0), turned to 90 degrees
- moved D2 117.7 mm to (176.5, 97.2)
- moved D9 117.2 mm to (173.0, 120.0), turned to 90 degrees
- moved D4 115.9 mm to (176.5, 102.5)
- moved D1 114.3 mm to (170.7, 97.2)
- moved D3 112.2 mm to (170.7, 102.5)
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Connections:
- U1 pad 19: /5V -> +5V
- U2 pad 11: unconnected-(U2-PD5-Pad11) -> /PD5
- U2 pad 12: unconnected-(U2-PD6-Pad12) -> /PD6
- U2 pad 13: unconnected-(U2-PD7-Pad13) -> /PD7
- U2 pad 14: unconnected-(U2-PB0-Pad14) -> /PB0
- U2 pad 15: unconnected-(U2-PB1-Pad15) -> /PB1
- U2 pad 2: unconnected-(U2-PD0-Pad2) -> /PD0
- U2 pad 23: unconnected-(U2-PC0-Pad23) -> +5V
- U2 pad 3: unconnected-(U2-PD1-Pad3) -> /PD1
- U2 pad 4: unconnected-(U2-PD2-Pad4) -> /PD2
- U2 pad 5: unconnected-(U2-PD3-Pad5) -> /PD3
- U2 pad 6: unconnected-(U2-PD4-Pad6) -> /PD4
- U2 pad 7: /5V -> +5V
Other:
- board size 136.8 x 99.6 mm -> 149.8 x 99.6 mm

Commit message: Auto stash before merge of "main" and "origin/main"
Routing:
- net /B: track 0.00 -> 449.7 mm
- net /A: track 0.00 -> 398.4 mm
- net /DP: track 0.00 -> 384.0 mm
- net GND: track 0.00 -> 326.0 mm
- net /DIG7: track 0.00 -> 318.6 mm
- net /F: track 0.00 -> 252.4 mm
- net +5V: track 0.00 -> 245.2 mm
- net /G: track 0.00 -> 243.0 mm
- net /PB1: track 0.00 -> 235.7 mm
- net /DIG5: track 0.00 -> 231.2 mm
- net /PB0: track 0.00 -> 212.6 mm
- net /E: track 0.00 -> 197.4 mm
- net /D: track 0.00 -> 170.9 mm
- net /C: track 0.00 -> 166.2 mm
- net /PD4: track 0.00 -> 120.5 mm
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
Commit message: kicad is done!
Parts:
- renumbered D1 to 1, D10 to 10, D11 to 11, D12 to 12, D13 to 13, D14 to 14, D15 to 15, D16 to 16, D2 to 2, D3 to 3, D4 to 4, D5 to 5, D6 to 6, D7 to 7, D8 to 8, D9 to 9
Routing:
- net /DIG4: track 7.62 -> 103.1 mm, vias 0 -> 5
- net /D: track 170.9 -> 255.0 mm, vias 0 -> 4
- net /E: track 197.4 -> 275.9 mm
- net /DIG1: track 7.62 -> 71.5 mm, vias 0 -> 3
- net /DIG6: track 69.3 -> 128.4 mm, vias 0 -> 1
- net MOSI: track 0.00 -> 59.1 mm, vias 0 -> 3
- net /C: track 166.2 -> 216.5 mm, vias 0 -> 2
- net SCK: track 54.0 -> 91.8 mm, vias 0 -> 1
- net MISO: track 0.00 -> 37.6 mm, vias 0 -> 1
- net /F: track 252.4 -> 288.3 mm, vias 0 -> 5
- net Net-(U1-ISET): track 0.00 -> 35.8 mm
- net /DIG0: track 73.6 -> 103.7 mm
- net +5V: track 245.2 -> 266.7 mm
- net /B: track 449.7 -> 470.5 mm
- net /A: track 398.4 -> 387.2 mm, vias 0 -> 1
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Other:
- board text added: "12.Ta två shots och hoppa på ett ben i 10 sekunder 13.Ta en {dblquote}grenad{dblquote} (shot + öl svep direkt efter varandra) 14.Byt ut din drink mot någon annans i nästa runda 15.Drick tre klunkar ur varje annan spelares drink 16.Halsa en öl och snurra 10 varv på stället 17.Drick upp det starkaste du hittar på bordet 18.Ta en shot och försök göra en kullerbytta 19.Häll upp tre shots - drick en o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"

Commit message: orded
Parts:
- removed 1, 10, 11, 12, 13, 14, 15, 16, 2, 3, 4, 5, 6, 7, 8, 9: LED, LED_THT:LED_D3.0mm_Clear
- removed RESET, WHEEL: SW_pin12, Button_Switch_THT:SW_PUSH-12mm_Wuerth-430476085716
- added D1: LED, LED_THT:LED_D3.0mm_Clear, F.Cu at (145.6, 97.3)
- added D10: LED, LED_THT:LED_D3.0mm_Clear, F.Cu at (147.2, 111.1)
- added D11: LED, LED_THT:LED_D3.0mm_Clear, F.Cu at (138.6, 102.9)
- added D12: LED, LED_THT:LED_D3.0mm_Clear, F.Cu at (138.6, 97.4)
- added D13: LED, LED_THT:LED_D3.0mm_Clear, F.Cu at (180.6, 86.1)
- added D14: LED, LED_THT:LED_D3.0mm_Clear, F.Cu at (186.1, 86.1)
- added D15: LED, LED_THT:LED_D3.0mm_Clear, F.Cu at (114.1, 86.1)
- added D16: LED, LED_THT:LED_D3.0mm_Clear, F.Cu at (119.6, 86.1)
- added D2: LED, LED_THT:LED_D3.0mm_Clear, F.Cu at (145.6, 102.7)
- added D3: LED, LED_THT:LED_D3.0mm_Clear, F.Cu at (151.7, 97.2)
- added D4: LED, LED_THT:LED_D3.0mm_Clear, F.Cu at (151.7, 102.7)
- added D5: LED, LED_THT:LED_D3.0mm_Clear, F.Cu at (147.7, 88.4)
- added D6: LED, LED_THT:LED_D3.0mm_Clear, F.Cu at (152.5, 88.5)
- added D7: LED, LED_THT:LED_D3.0mm_Clear, F.Cu at (162.5, 96.0)
- added D8: LED, LED_THT:LED_D3.0mm_Clear, F.Cu at (162.5, 101.5)
- added D9: LED, LED_THT:LED_D3.0mm_Clear, F.Cu at (152.7, 111.1)
- added SW3: SW_pin12, Button_Switch_THT:SW_PUSH-12mm_Wuerth-430476085716, F.Cu at (142.8, 120.7)
- added SW4: SW_pin12, Button_Switch_THT:SW_PUSH-12mm_Wuerth-430476085716, F.Cu at (162.9, 130.2)
- moved U2 113.6 mm to (138.3, 143.2)
- moved U7 98.0 mm to (122.2, 91.2), turned to -90 degrees
- moved U8 97.7 mm to (122.2, 102.1), turned to -90 degrees
- moved U1 96.6 mm to (160.8, 151.5), turned to 90 degrees
- moved J5 91.4 mm to (147.8, 155.7)
- moved J6 76.2 mm to (182.7, 132.0), turned to 0 degrees
- moved U9 73.1 mm to (113.2, 123.8), turned to 0 degrees
- moved R1 71.2 mm to (145.0, 131.3), turned to 0 degrees
- moved U6 58.8 mm to (178.1, 98.7)
- moved U5 58.7 mm to (178.1, 109.6)
- moved U10 51.7 mm to (124.5, 123.7), turned to 0 degrees
- moved J3 51.7 mm to (195.8, 94.4), turned to 0 degrees
- moved R2 33.9 mm to (145.0, 134.5)
- moved R3 22.5 mm to (145.0, 137.7)
- moved J4 2.04 mm to (102.5, 94.4)
Routing:
- net /B: track 470.5 -> 175.2 mm
- net /PB1: track 235.7 -> 45.7 mm
- net /PB0: track 207.1 -> 47.7 mm
- net /DP: track 394.9 -> 239.3 mm, vias 2 -> 6
- net /DIG5: track 231.2 -> 75.5 mm, vias 0 -> 2
- net /DIG7: track 320.2 -> 169.0 mm, vias 0 -> 11
- net /A: track 387.2 -> 236.6 mm, vias 1 -> 0
- net +5V: track 266.7 -> 139.9 mm, vias 0 -> 9
- net MISO: track 37.6 -> 145.2 mm, vias 1 -> 2
- net /PD1: track 68.6 -> 174.6 mm
- net GND: track 326.0 -> 235.2 mm, vias 0 -> 5
- net /G: track 245.6 -> 162.9 mm
- net /PD7: track 110.2 -> 43.3 mm
- net /PD6: track 111.1 -> 46.9 mm
- net /PD5: track 112.1 -> 50.5 mm
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Other:
- board size 149.8 x 99.6 mm -> 99 x 99 mm
- board text added: "Bobo Bäck Engström Think Fast"
- board text removed: "12.Ta två shots och hoppa på ett ben i 10 sekunder 13.Ta en {dblquote}grenad{dblquote} (shot + öl svep direkt efter varandra) 14.Byt ut din drink mot någon annans i nästa runda 15.Drick tre klunkar ur varje annan spelares drink 16.Halsa en öl och snurra 10 varv på stället 17.Drick upp det starkaste du hittar på bordet 18.Ta en shot och försök göra en kullerbytta 19.Häll upp tre shots - drick en o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"
