File: kicad/Game_project/game.kicad_sch (KiCad schematic)
At the start: 27 parts, among them J5 USB_B, J6 ISP header, U1 MAX7219, U10 HDSP-7403, U2 ATmega328P-P, U5 HDSP-7403, U6 HDSP-7403, U7 HDSP-7403, U8 HDSP-7403, U9 HDSP-7403

Commit message: new kicad
Other:
- note removed: "* Indicates a PWM-capable pin"
- moved on the sheet: D1, D10, D11, D12, D13, D14, D15, D16, D2, D3, D4, D5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

Commit message: snart klar i kicad de ska bara rotas
Parts:
- added J3, J4: Conn_01x05_Socket, Connector_PinSocket_2.54mm:PinSocket_1x05_P2.54mm_Vertical, symbol Connector:Conn_01x05_Socket
- added R2, R3: 10k, Resistor_THT:R_Axial_DIN0204_L3.6mm_D1.6mm_P7.62mm_Horizontal, symbol Device:R
- added SW3, SW4: SW_pin12, Button_Switch_THT:SW_PUSH-12mm_Wuerth-430476085716, symbol Switch:SW_MEC_5E
- U1: footprint Package_DIP:DIP-24_18.0mmx34.29mm_W15.24mm -> Package_DIP:DIP-28_W7.62mm
Connections:
- net 5V is gone; now on net +5V: U1.19 (V+), U2.7 (VCC)
- net +5V: now also U2.23 (PC0), SW3.1, SW4.1
- net GND: now also J3.5 (Pin_5), J4.5 (Pin_5), R2.2, R3.2
- net PD5: now reaches U2.11 (PD5)
- net PD5: now also J4.2 (Pin_2)
- net PD6: now reaches U2.12 (PD6)
- net PD6: now also J4.3 (Pin_3)
- net PD7: now reaches U2.13 (PD7)
- net PD7: now also J4.4 (Pin_4)
- net PB0: now reaches U2.14 (PB0)
- net PB0: now also R2.1, SW3.4 (A)
- net PB1: now reaches U2.15 (PB1)
- net PB1: now also R3.1, SW4.4 (A)
- net PD0: now reaches U2.2 (PD0)
- net PD0: now also J3.1 (Pin_1)
- net PD1: now reaches U2.3 (PD1)
- net PD1: now also J3.2 (Pin_2)
- net PD2: now reaches U2.4 (PD2)
- net PD2: now also J3.3 (Pin_3)
- net PD3: now reaches U2.5 (PD3)
- net PD3: now also J3.4 (Pin_4)
- net PD4: now reaches U2.6 (PD4)
- net PD4: now also J4.1 (Pin_1)
- no-connect marks 0 -> 4

Commit message: orded
Parts:
- R1: value 10k -> 50k
Connections:
- no-connect marks 4 -> 5

Commit message: find wrong
Connections:
- net F: no longer D15.2 (A), D7.2 (A)
- net G: now also D15.2 (A), D7.2 (A)
Changed lines of the file:
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@@
+		)
+	)
+	(label "G"
+		(at 246.38 66.04 0)
+		(effects
+			(font
+				(size 1.27 1.27)
+			)
+			(justify left bottom)
+		)
+	)
+	(label "G"
+		(at 274.32 66.04 0)
+		(effects
+			(font
+				(size 1.27 1.27)
+			)
+			(justify left bottom)
 		)
 	)
@@
 		)
 	)
-	(label "F"
-		(at 274.32 66.04 0)
-		(effects
-			(font
-				(size 1.27 1.27)
-			)
-			(justify left bottom)
-		)
-	)
 	(label "A"
 		(at 166.37 66.04 0)
@@
 		(effects
 			(font
-				(size 1.27 1.27)
-			)
-			(justify left bottom)
-		)
-	)
-	(label "F"
-		(at 246.38 66.04 0)
-		(effects
-			(font
